File: explorations/MC6809_SBC1/MC6809_SBC1/MC6809_SBC1.kicad_sch (KiCad schematic)
At the start: 11 parts, among them U1 MC6809, Y1 3.6864 MHz

Commit message: SBC1 scheme a& other stuff
Parts:
- added C11, C12, C13, C14: 100n, Capacitor_THT:C_Disc_D3.0mm_W1.6mm_P2.50mm, symbol Device:C
- added C15: 10u, symbol Device:C_Polarized
- added D1: 1N4148, Diode_THT:D_DO-35_SOD27_P7.62mm_Horizontal, symbol Diode:1N4148
- added J1: Serial, symbol Connector:Conn_01x06_Pin
- added R23: 2K2, Resistor_THT:R_Axial_DIN0207_L6.3mm_D2.5mm_P7.62mm_Horizontal, symbol Device:R
- added SW1: V, symbol Switch:SW_Push
- added U4: MC68B50, Package_DIP:DIP-24_W15.24mm, symbol Interface_UART:MC68B50
- added U5: 27C512, Package_DIP:DIP-28_W15.24mm, symbol Memory_EPROM:27C512
- added U6: HM62256BLP, Package_DIP:DIP-28_W15.24mm, symbol Memory_RAM:HM62256BLP
- added U7: 74LS00, symbol 74xx:74LS00
- C1, C2: value 15p -> 24p
Connections:
- net GND: now also C11.1, C12.1, C13.1, C14.1, C15.2, J1.6 (Pin_6), SW1.1, U4.1 (VSS), U4.23 (~{DCD}), U5.1 (A15), U5.14 (GND), U5.27 (A14), U6.14 (GND), U7.7 (GND)
- net IRQ_: now also U4.7 (~{IRQ})
- net VCC: now also C11.2, C12.2, C13.2, C14.2, D1.1 (K), R23.1, U4.12 (VCC), U5.28 (VCC), U6.28 (VCC), U7.14 (VCC)
- net A2: now reaches U1.10 (A2)
- net A2: now also U5.8 (A2), U6.8 (A2)
- net A3: now reaches U1.11 (A3)
- net A3: now also U5.7 (A3), U6.7 (A3)
- net A4: now reaches U1.12 (A4)
- net A4: now also U5.6 (A4), U6.6 (A4)
- net A5: now reaches U1.13 (A5)
- net A5: now also U5.5 (A5), U6.5 (A5)
- net A6: now reaches U1.14 (A6)
- net A6: now also U5.4 (A6), U6.4 (A6)
- net A7: now reaches U1.15 (A7)
- net A7: now also U5.3 (A7), U6.3 (A7)
- net A8: now reaches U1.16 (A8)
- net A8: now also U5.25 (A8), U6.25 (A8)
- net A9: now reaches U1.17 (A9)
- net A9: now also U5.24 (A9), U6.24 (A9)
- net A10: now reaches U1.18 (A10)
- net A10: now also U5.21 (A10), U6.21 (A10)
- net A11: now reaches U1.19 (A11)
- net A11: now also U5.23 (A11), U6.23 (A11)
- net A12: now reaches U1.20 (A12)
- net A12: now also U5.2 (A12), U6.2 (A12)
- net A13: now reaches U1.21 (A13)
- net A13: now also U4.10 (CS1), U5.26 (A13), U6.26 (A13)
- net A14: now reaches U1.22 (A14)
- net A14: now also U4.9 (CS2), U6.1 (A14), U7.1
- net A15: now reaches U1.23 (A15)
- net A15: now also U4.8 (CS0), U6.20 (~{CS}), U7.2
- net D7: now reaches U1.24 (D7)
- net D7: now also U4.15 (D7), U5.19 (D7), U6.19 (Q7)
- net D6: now reaches U1.25 (D6)
- net D6: now also U4.16 (D6), U5.18 (D6), U6.18 (Q6)
- net D5: now reaches U1.26 (D5)
- net D5: now also U4.17 (D5), U5.17 (D5), U6.17 (Q5)
- net D4: now reaches U1.27 (D4)
- net D4: now also U4.18 (D4), U5.16 (D4), U6.16 (Q4)
- net D3: now reaches U1.28 (D3)
- net D3: now also U4.19 (D3), U5.15 (D3), U6.15 (Q3)
- net D2: now reaches U1.29 (D2)
- net D2: now also U4.20 (D2), U5.13 (D2), U6.13 (Q2)
- net D1: now reaches U1.30 (D1)
- net D1: now also U4.21 (D1), U5.12 (D1), U6.12 (Q1)
- net D0: now reaches U1.31 (D0)
- net D0: now also U4.22 (D0), U5.11 (D0), U6.11 (Q0)
- net RW: now reaches U1.32 (R/~{W})
- net RW: now also U7.12, U7.13, U7.4
- net E: now reaches U1.34 (E)
- net E: now also U4.14 (E), U4.3 (Rx_CLK), U4.4 (Tx_CLK), U7.5, U7.9
- net at U1.37 (~{RESET}): now also C15.1, D1.2 (A), R23.2, SW1.2
- net A0: now reaches U1.8 (A0)
- net A0: now also U4.11 (RS), U5.10 (A0), U6.10 (A0)
- net A1: now reaches U1.9 (A1)
- net A1: now also U5.9 (A1), U6.9 (A1)
- new net: J1.2 (Pin_2), U4.6 (Tx_Data)
- new net: J1.3 (Pin_3), U4.2 (Rx_Data)
- new net: U7.10, U7.11
- new net: U4.24 (~{CTS}), U4.5 (~{RTS})
- new net READ: U5.22 (~{OE}), U6.22 (~{OE}), U7.6
- new net ROM_CS: U5.20 (~{CE}), U7.3
- new net WRITE: U6.27 (~{WE}), U7.8
Other:
- note added: "0000-7FFF : 32K RAM 8000-9FFF : 8K NOT USED A000-BFFF : 8K MC6850 C000-FFFF : 16K ROM"
- note added: "Changes: the EEPROM used is the W27C512 (64K Bytes)"
- note added: "FTDI"
- note added: "Free Run & Clock with inductor Not required"
- note added: "MC6809P SBC1, credits to Searle Grant and Jeff Tranter."
- note added: "Memory Map"
- note added: "RAM_CS = A15"
- note added: "the CPU is MC6809P, not the MC68B09P, and the clock is 3.6864 Mhz (require 24p capacitors)"
- moved on the sheet: C1, C2, C9, U1, Y1
